File: .history/power.kicad_sch (KiCad schematic)
At the start: 17 parts, among them J1 Conn_02x08_Odd_Even, U1 TL072

Commit message: adding values to caps
Parts:
- U1: footprint (none) -> Package_SO:SOIC-8_3.9x4.9mm_P1.27mm
- renumbered C1 to C11, C4 to C12, C2 to C13, C5 to C14, C3 to C15, C6 to C16, C7 to C17, C8 to C18, J1 to J5, TP1 to TP2, TP2 to TP3, TP3 to TP4, TP4 to TP5
Changed lines of the file:
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@@
 		(in_pos_files yes)
 		(dnp no)
-		(property "Reference" "TP2"
+		(property "Reference" "TP3"
 			(at 143.002 52.07 0)
 			(show_name no)
@@
 			(project "Arduino VCO"
 				(path "/3a28b572-943c-402b-9245-b62f72b0a8e3/6ad9a068-c00b-4d78-a509-b3a18517b3c8"
-					(reference "TP2")
+					(reference "TP3")
 					(unit 1)
 				)
@@
 		(in_pos_files yes)
 		(dnp no)
-		(property "Reference" "C4"
+		(property "Reference" "C12"
 			(at 124.714 40.64 0)
 			(show_name no)
@@
 			(project "Arduino VCO"
 				(path "/3a28b572-943c-402b-9245-b62f72b0a8e3/6ad9a068-c00b-4d78-a509-b3a18517b3c8"
-					(reference "C4")
+					(reference "C12")
 					(unit 1)
 				)
@@
 		(dnp no)
 		(fields_autoplaced yes)
-		(property "Reference" "#PWR031"
+		(property "Reference" "#PWR040"
 			(at 26.67 123.19 0)
 			(hide yes)
@@
 			(project "Arduino VCO"
 				(path "/3a28b572-943c-402b-9245-b62f72b0a8e3/6ad9a068-c00b-4d78-a509-b3a18517b3c8"
-					(reference "#PWR031")
+					(reference "#PWR040")
 					(unit 1)
 				)
@@
 		(in_pos_files yes)
 		(dnp no)
-		(property "Reference" "C5"
+		(property "Reference" "C14"
 			(at 124.714 63.5 0)
 			(show_name no)
@@
 			(project "Arduino VCO"
 				(path "/3a28b572-943c-402b-9245-b62f72b0a8e3/6ad9a068-c00b-4d78-a509-b3a18517b3c8"
-					(reference "C5")
+					(reference "C14")
 					(unit 1)
 				)
@@
 		(dnp no)
 		(fields_autoplaced yes)
-		(property "Reference" "#PWR04"
+		(property "Reference" "#PWR038"
 			(at 152.4 76.2 0)
 			(hide yes)
@@
 			(project "Arduino VCO"
 				(path "/3a28b572-943c-402b-9245-b62f72b0a8e3/6ad9a068-c00b-4d78-a509-b3a18517b3c8"
-					(reference "#PWR04")
+					(reference "#PWR038")
 					(unit 1)
 				)
@@
 		(dnp no)
 		(fields_autoplaced yes)
-		(property "Reference" "#PWR030"
+		(property "Reference" "#PWR041"
 			(at 54.61 125.73 0)
 			(hide yes)
@@
 			(project "Arduino VCO"
 				(path "/3a28b572-943c-402b-9245-b62f72b0a8e3/6ad9a068-c00b-4d78-a509-b3a18517b3c8"
-					(reference "#PWR030")
+					(reference "#PWR041")
 					(unit 1)
 				)
@@
 		(in_pos_files yes)
 		(dnp no)
-		(property "Reference" "#PWR03"
+		(property "Reference" "#PWR037"
 			(at 152.4 77.47 0)
 			(hide yes)
@@
 			(project "Arduino VCO"
 				(path "/3a28b572-943c-402b-9245-b62f72b0a8e3/6ad9a068-c00b-4d78-a509-b3a18517b3c8"
-					(reference "#PWR03")
+					(reference "#PWR037")
 					(unit 1)
 				)
@@
 		(in_pos_files yes)
 		(dnp no)
-		(property "Reference" "TP3"
+		(property "Reference" "TP4"
 			(at 143.002 63.754 0)
 			(show_name no)
@@
 			(project "Arduino VCO"
 				(path "/3a28b572-943c-402b-9245-b62f72b0a8e3/6ad9a068-c00b-4d78-a509-b3a18517b3c8"
-					(reference "TP3")
+					(reference "TP4")
 					(unit 1)
 				)
@@
 		(in_pos_files yes)
 		(dnp no)
-		(property "Reference" "C3"
+		(property "Reference" "C15"
 			(at 110.744 73.66 0)
 			(show_name no)
@@
 			(project "Arduino VCO"
 				(path "/3a28b572-943c-402b-9245-b62f72b0a8e3/6ad9a068-c00b-4d78-a509-b3a18517b3c8"
-					(reference "C3")
+					(reference "C15")
 					(unit 1)
 				)
@@
 		(in_pos_files yes)
 		(dnp no)
-		(property "Reference" "C1"
+		(property "Reference" "C11"
 			(at 110.998 40.64 0)
 			(show_name no)
@@
 			(project "Arduino VCO"
 				(path "/3a28b572-943c-402b-9245-b62f72b0a8e3/6ad9a068-c00b-4d78-a509-b3a18517b3c8"
-					(reference "C1")
+					(reference "C11")
 					(unit 1)
 				)
@@
 		(in_pos_files yes)
 		(dnp no)
-		(property "Reference" "C7"
+		(property "Reference" "C17"
 			(at 49.784 110.236 0)
 			(show_name no)
@@
 			(project "Arduino VCO"
 				(path "/3a28b572-943c-402b-9245-b62f72b0a8e3/6ad9a068-c00b-4d78-a509-b3a18517b3c8"
-					(reference "C7")
+					(reference "C17")
 					(unit 1)
 				)
@@
 		(in_pos_files yes)
 		(dnp no)
-		(property "Reference" "#PWR07"
+		(property "Reference" "#PWR034"
 			(at 152.4 55.88 0)
 			(hide yes)
@@
 			(project "Arduino VCO"
 				(path "/3a28b572-943c-402b-9245-b62f72b0a8e3/6ad9a068-c00b-4d78-a509-b3a18517b3c8"
-					(reference "#PWR07")
+					(reference "#PWR034")
 					(unit 1)
 				)
@@
 		(in_pos_files yes)
 		(dnp no)
-		(property "Reference" "#PWR02"
+		(property "Reference" "#PWR035"
 			(at 152.4 62.23 0)
 			(hide yes)
@@
 			(project "Arduino VCO"
 				(path "/3a28b572-943c-402b-9245-b62f72b0a8e3/6ad9a068-c00b-4d78-a509-b3a18517b3c8"
-					(reference "#PWR02")
+					(reference "#PWR035")
 					(unit 1)
 				)
@@
 		(dnp no)
 		(fields_autoplaced yes)
-		(property "Reference" "#PWR05"
+		(property "Reference" "#PWR033"
 			(at 152.4 39.37 0)
 			(hide yes)
@@
 			(project "Arduino VCO"
 				(path "/3a28b572-943c-402b-9245-b62f72b0a8e3/6ad9a068-c00b-4d78-a509-b3a18517b3c8"
-					(reference "#PWR05")
+					(reference "#PWR033")
 					(unit 1)
 				)
@@
 		(in_pos_files yes)
 		(dnp no)
-		(property "Reference" "J1"
+		(property "Reference" "J5"
 			(at 45.974 78.232 0)
 			(show_name no)
@@
 			(project "Arduino VCO"
 				(path "/3a28b572-943c-402b-9245-b62f72b0a8e3/6ad9a068-c00b-4d78-a509-b3a18517b3c8"
-					(reference "J1")
+					(reference "J5")
 					(unit 1)
 				)
@@
 		(in_pos_files yes)
 		(dnp no)
-		(property "Reference" "C6"
+		(property "Reference" "C16"
 			(at 124.714 73.406 0)
 			(show_name no)
@@
 			(project "Arduino VCO"
 				(path "/3a28b572-943c-402b-9245-b62f72b0a8e3/6ad9a068-c00b-4d78-a509-b3a18517b3c8"
-					(reference "C6")
+					(reference "C16")
 					(unit 1)
 				)
@@
 		(in_pos_files yes)
 		(dnp no)
-		(property "Reference" "TP4"
+		(property "Reference" "TP5"
 			(at 143.256 74.676 0)
 			(show_name no)
@@
 			(project "Arduino VCO"
 				(path "/3a28b572-943c-402b-9245-b62f72b0a8e3/6ad9a068-c00b-4d78-a509-b3a18517b3c8"
-					(reference "TP4")
+					(reference "TP5")
 					(unit 1)
 				)
@@
 		(in_pos_files yes)
 		(dnp no)
-		(property "Reference" "TP1"
+		(property "Reference" "TP2"
 			(at 137.414 27.686 0)
 			(show_name no)
@@
 			(project "Arduino VCO"
 				(path "/3a28b572-943c-402b-9245-b62f72b0a8e3/6ad9a068-c00b-4d78-a509-b3a18517b3c8"
-					(reference "TP1")
+					(reference "TP2")
 					(unit 1)
 				)
@@
 		(in_pos_files yes)
 		(dnp no)
-		(property "Reference" "#PWR01"
+		(property "Reference" "#PWR036"
 			(at 29.21 71.12 0)
 			(hide yes)
@@
 			(project "Arduino VCO"
 				(path "/3a28b572-943c-402b-9245-b62f72b0a8e3/6ad9a068-c00b-4d78-a509-b3a18517b3c8"
-					(reference "#PWR01")
+					(reference "#PWR036")
 					(unit 1)
 				)
@@
 		(in_pos_files yes)
 		(dnp no)
-		(property "Reference" "#FLG02"
+		(property "Reference" "#FLG01"
 			(at 96.52 56.515 0)
 			(hide yes)
@@
 			(project "Arduino VCO"
 				(path "/3a28b572-943c-402b-9245-b62f72b0a8e3/6ad9a068-c00b-4d78-a509-b3a18517b3c8"
-					(reference "#FLG02")
+					(reference "#FLG01")
 					(unit 1)
 				)
@@
 			)
 		)
-		(property "Footprint" ""
+		(property "Footprint" "Package_SO:SOIC-8_3.9x4.9mm_P1.27mm"
 			(at 57.15 116.84 0)
 			(hide yes)
@@
 		(dnp no)
 		(fields_autoplaced yes)
-		(property "Reference" "#PWR029"
+		(property "Reference" "#PWR039"
 			(at 54.61 107.95 0)
 			(hide yes)
@@
 			(project "Arduino VCO"
 				(path "/3a28b572-943c-402b-9245-b62f72b0a8e3/6ad9a068-c00b-4d78-a509-b3a18517b3c8"
-					(reference "#PWR029")
+					(reference "#PWR039")
 					(unit 1)
 				)
@@
 		(dnp no)
 		(fields_autoplaced yes)
-		(property "Reference" "#FLG01"
+		(property "Reference" "#FLG02"
 			(at 30.48 61.595 0)
 			(hide yes)
@@
 			(project "Arduino VCO"
 				(path "/3a28b572-943c-402b-9245-b62f72b0a8e3/6ad9a068-c00b-4d78-a509-b3a18517b3c8"
-					(reference "#FLG01")
+					(reference "#FLG02")
 					(unit 1)
 				)
@@
 		(in_pos_files yes)
 		(dnp no)
-		(property "Reference" "C2"
+		(property "Reference" "C13"
 			(at 110.998 63.5 0)
 			(show_name no)
@@
 			(project "Arduino VCO"
 				(path "/3a28b572-943c-402b-9245-b62f72b0a8e3/6ad9a068-c00b-4d78-a509-b3a18517b3c8"
-					(reference "C2")
+					(reference "C13")
 					(unit 1)
 				)
@@
 		(in_pos_files yes)
 		(dnp no)
-		(property "Reference" "C8"
+		(property "Reference" "C18"
 			(at 50.038 120.65 0)
 			(show_name no)
@@
 			(project "Arduino VCO"
 				(path "/3a28b572-943c-402b-9245-b62f72b0a8e3/6ad9a068-c00b-4d78-a509-b3a18517b3c8"
-					(reference "C8")
-					(unit 1)
-				)
+					(reference "C18")
+					(unit 1)
+				)
