File: Electronics/Arduino VCO.kicad_sch (KiCad schematic)
At the start: 63 parts, among them SW1 MODE, U1 TL072

Commit message: starting pcb
Parts:
- removed C10: 10uF, Capacitor_SMD:CP_Elec_5x5.4, symbol Device:C_Polarized
- removed C9: 100nF, Capacitor_SMD:C_0805_2012Metric_Pad1.18x1.45mm_HandSolder, symbol Device:C
- removed TP1: A, TestPoint:TestPoint_Pad_D1.5mm, symbol Connector:TestPoint
- D6, D7, D8: footprint LED_THT:LED_D3.0mm_IRBlack -> LED_THT:LED_D3.0mm_Clear
- SW1: footprint Button_Switch_THT:SW_PUSH_6mm -> Button_Switch_THT:SW_PUSH_6mm_H13mm

Commit message: finishing tracks and resolving drc errors
Parts:
- SW1: footprint Button_Switch_THT:SW_PUSH_6mm_H13mm -> Eurorack:SW_PUSH_6mm_H13mm_1
Changed lines of the file:
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@@
 			)
 		)
-		(property "Footprint" "Button_Switch_THT:SW_PUSH_6mm_H13mm"
+		(property "Footprint" "Eurorack:SW_PUSH_6mm_H13mm_1"
 			(at 184.15 34.29 0)
 			(hide yes)

Commit message: Adding Silkscreen symbols
Other:
- company: ©Dirty Dream - Nathanael Noir -> © Dirty Dream – Nathanael Noir
Changed lines of the file:
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@@
 	(title_block
 		(title "CY3-FOLD VCO")
-		(date "2026-04-17")
+		(date "2026-06-21")
 		(rev "v1.0")
-		(company "©Dirty Dream - Nathanael Noir")
+		(company "© Dirty Dream – Nathanael Noir")
 	)
 	(rectangle
